File: necpc8801mkiisr.sch (KiCad schematic (older format))
At the start: 232 parts, among them J1 Conn_01x04_MountingPin, SW1 SW_Push, U1 ATmega32U4-AU, Y1 16MHz

Commit message: fix
Parts:
- SW_0, SW_1, SW_2, SW_3, SW_4, SW_5, SW_6, SW_7, SW_8, SW_9, SW_A1, SW_APOS1, SW_B1, SW_BACKSP1, SW_BKSLS1, SW_C1, SW_CAP1, SW_COLON1, SW_COMMA1, SW_D1, SW_DEL1, SW_DOWN1, SW_E1, SW_END1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: value MX-NoLED -> mx-alps-fut; symbol MX_Alps_Hybrid:MX-NoLED -> MX_Alps_Hybrid:mx-alps-fut
