File: necpc8801mkiisr.kicad_sch (KiCad schematic)
At the start: 217 parts, among them J1 Conn_01x04_MountingPin, SW1 SW_Push, U1 ATmega32U4-MU, Y1 16MHz

Commit message: fix
Parts:
- removed SW_RSH_ALIAS_1: MX-NoLED, MX_NEC:mx-nec-alps, symbol MX_Alps_Hybrid:MX-NoLED
Connections:
- net COL0: now also U1.27 (PD7); no longer U1.41 (PF0)
- net COL1: now also U1.28 (PB4); no longer U1.36 (PF7)
- net COL2: now also U1.29 (PB5); no longer U1.38 (PF5)
- net COL3: now also U1.30 (PB6); no longer U1.37 (PF6)
- net COL4: now also U1.32 (PC7); no longer U1.39 (PF4)
- net COL5: now also U1.36 (PF7); no longer U1.27 (PD7)
- net COL6: now also U1.37 (PF6); no longer U1.29 (PB5)
- net COL7: now also U1.38 (PF5); no longer U1.30 (PB6)
- net COL9: now also U1.22 (PD5); no longer U1.8 (PB0)
- net ROW0: now also U1.12 (PB7); no longer U1.40 (PF1)
- net ROW1: now also U1.10 (PB2); no longer U1.11 (PB3)
- net ROW2: now also U1.8 (PB0); no longer U1.12 (PB7)
- net ROW3: now also U1.18 (PD0); no longer U1.28 (PB4)
- net ROW4: now also U1.26 (PD6); no longer U1.22 (PD5)
- net ROW6: now also U1.19 (PD1); no longer U1.26 (PD6)
- net ROW7: now also U1.39 (PF4); no longer U1.19 (PD1)
- net ROW8: now also U1.41 (PF0); no longer U1.18 (PD0)
- net ROW9: now also U1.11 (PB3); no longer U1.10 (PB2)
- net ROW10: no longer names the net of U1.9 (PB1)

Commit message: update
Parts:
- SW_0_1, SW_1_1, SW_2_1, SW_3_1, SW_4_1, SW_5_1, SW_6_1, SW_7_1, SW_8_1, SW_9_1, SW_ALT_1, SW_AMG_1, SW_AT_1, SW_A_1, SW_B_1, SW_CAPS_1, SW_CAR_1, SW_COL_1, SW_CPY_1, SW_CTRL_1, SW_C_1, SW_DEL_1, SW_DOWN_1, SW_D_1, SW_ED_1, SW_ESC_1, SW_ET_1, SW_E_1, SW_F1_1, SW_F2_1, SW_F3_1, SW_F4_1, SW_F5_1, SW_FC_1, SW_F_1, SW_GT_1, SW_G_1, SW_H_1, SW_I_1, SW_J_1, SW_KP0_1, SW_KP1_1, SW_KP2_1, SW_KP3_1, SW_KP4_1, SW_KP5_1, SW_KP6_1, SW_KP7_1, SW_KP8_1, SW_KP9_1, SW_KPCOM_1, SW_KPDIV_1, SW_KPENT_1, SW_KPEQ_1, SW_KPHELP1, SW_KPHOME_1, SW_KPMIN_1, SW_KPMULT_1, SW_KPPER_1, SW_KPPLUS_1, SW_K_1, SW_LEFT_1, SW_LS1_1, SW_LS2_1, SW_LT_1, SW_L_1, SW_MN_1, SW_M_1, SW_N_1, SW_O_1, SW_P_1, SW_Q_1, SW_RIGHT_1, SW_RLD_1, SW_RLU_1, SW_RSH_1, SW_R_1, SW_SLS_1, SW_SMI_1, SW_SP1_1, SW_SP2_1, SW_STP_1, SW_SUP_1, SW_S_1, SW_TAB_1, SW_T_1, SW_UP_1, SW_U_1, SW_V_1, SW_WE_1, SW_W_1, SW_X_1, SW_YEN_1, SW_Y_1, SW_Z_1: footprint MX_NEC:mx-nec-alps -> MX_NEC:mx-alps-futaba

Commit message: fix
Parts:
- SW_0_1, SW_1_1, SW_2_1, SW_3_1, SW_4_1, SW_5_1, SW_6_1, SW_7_1, SW_8_1, SW_9_1, SW_ALT_1, SW_AMG_1, SW_AT_1, SW_A_1, SW_B_1, SW_CAPS_1, SW_CAR_1, SW_COL_1, SW_CPY_1, SW_CTRL_1, SW_C_1, SW_DEL_1, SW_DOWN_1, SW_D_1, SW_ED_1, SW_ESC_1, SW_ET_1, SW_E_1, SW_F1_1, SW_F2_1, SW_F3_1, SW_F4_1, SW_F5_1, SW_FC_1, SW_F_1, SW_GT_1, SW_G_1, SW_H_1, SW_I_1, SW_J_1, SW_KP0_1, SW_KP1_1, SW_KP2_1, SW_KP3_1, SW_KP4_1, SW_KP5_1, SW_KP6_1, SW_KP7_1, SW_KP8_1, SW_KP9_1, SW_KPCOM_1, SW_KPDIV_1, SW_KPENT_1, SW_KPEQ_1, SW_KPHELP1, SW_KPHOME_1, SW_KPMIN_1, SW_KPMULT_1, SW_KPPER_1, SW_KPPLUS_1, SW_K_1, SW_LEFT_1, SW_LS1_1, SW_LS2_1, SW_LT_1, SW_L_1, SW_MN_1, SW_M_1, SW_N_1, SW_O_1, SW_P_1, SW_Q_1, SW_RIGHT_1, SW_RLD_1, SW_RLU_1, SW_RSH_1, SW_R_1, SW_SLS_1, SW_SMI_1, SW_SP1_1, SW_SP2_1, SW_STP_1, SW_SUP_1, SW_S_1, SW_TAB_1, SW_T_1, SW_UP_1, SW_U_1, SW_V_1, SW_WE_1, SW_W_1, SW_X_1, SW_YEN_1, SW_Y_1, SW_Z_1: value MX-NoLED -> mx-alps-fut; symbol MX_Alps_Hybrid:MX-NoLED -> MX_Alps_Hybrid:mx-alps-fut

Commit message: updates
Connections:
- net ROW2: now also U1.11 (PB3); no longer U1.8 (PB0)
- net ROW9: now also U1.8 (PB0); no longer U1.11 (PB3)
Changed lines of the file:
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@@
     (effects (font (size 1.27 1.27)) (justify left bottom))
   )
-  (global_label "ROW2" (shape input) (at 81.28 49.53 0) (fields_autoplaced)
+  (global_label "ROW2" (shape input) (at 81.28 57.15 0) (fields_autoplaced)
     (effects (font (size 1.27 1.27)) (justify left))
-    (property "Intersheetrefs" "${INTERSHEET_REFS}" (at 1.27 -54.61 0)
+    (property "Intersheetrefs" "${INTERSHEET_REFS}" (at 1.27 -46.99 0)
       (effects (font (size 1.27 1.27)) hide)
     )
@@
     )
   )
-  (global_label "ROW9" (shape input) (at 81.28 57.15 0) (fields_autoplaced)
+  (global_label "ROW9" (shape input) (at 81.28 49.53 0) (fields_autoplaced)
     (effects (font (size 1.27 1.27)) (justify left))
-    (property "Intersheetrefs" "${INTERSHEET_REFS}" (at 1.27 -77.47 0)
+    (property "Intersheetrefs" "${INTERSHEET_REFS}" (at 1.27 -85.09 0)
       (effects (font (size 1.27 1.27)) hide)
     )
